Commit message: chore: Update robot.urdf with laser frame link and base to laser joint

File: urdf/robot.urdf (robot description, URDF)
Before this commit: robot simple_robot, 1 links, 1 joints
Links:
- added link laser_frame
Joints:
- removed joint fixed_joint
- added joint base_to_laser: type fixed, parent base_link, child laser_frame, origin xyz=0 0 0.2 rpy=0 0 0
